File: BreadBoard PS Fixed 5V/BreadBoard PS Ver2.kicad_pcb (KiCad board)
At the start: 2 copper layers, 29.8 x 52 mm, 15 parts, among them J1 Barrel_Jack_Switch_MountingPin, J2 Conn_02x02_Odd_Even, J3 Conn_02x02_Odd_Even, J4 Conn_02x02_Odd_Even, J5 Conn_02x02_Odd_Even, SW1 SW_DPDT_x2, U1 LM7805_TO220

Commit message: PCB wiring
Routing:
- net /Gnd: track 0.00 -> 98.3 mm
- net /5V-out: track 0.00 -> 84.1 mm
- net /5V: track 0.00 -> 45.3 mm
- net Net-(D3-Pad2): track 0.00 -> 36.1 mm
- net /Vin: track 0.00 -> 34.0 mm
- net Net-(D5-Pad1): track 0.00 -> 24.9 mm
- net Net-(D1-Pad2): track 0.00 -> 23.6 mm
Changed lines of the file:
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@@
     (thickness 1.6)
     (drawings 11)
-    (tracks 0)
+    (tracks 86)
     (zones 0)
     (modules 15)
@@
   )
   (setup
-    (last_trace_width 0.25)
+    (last_trace_width 0.3)
     (user_trace_width 0.3)
     (trace_clearance 0.2)
@@
     (solder_mask_min_width 0.25)
     (aux_axis_origin 0 0)
-    (visible_elements FFFFFF7F)
+    (visible_elements 7FFFFFFF)
     (pcbplotparams
       (layerselection 0x010fc_ffffffff)
@@
   (gr_arc (start 167.3225 75.6793) (end 167.3225 72.0725) (angle 90) (layer Edge.Cuts) (width 0.05))
   (gr_arc (start 167.3225 120.4341) (end 167.3225 124.0409) (angle -90) (layer Edge.Cuts) (width 0.05))
+  (segment (start 162.3695 108.4915) (end 162.3695 109.7915) (width 0.3) (layer F.Cu) (net 1))
+  (segment (start 156.5702 102.6922) (end 162.3695 108.4915) (width 0.3) (layer F.Cu) (net 1))
+  (segment (start 150.911 102.6922) (end 156.5702 102.6922) (width 0.3) (layer F.Cu) (net 1))
+  (segment (start 150.911 90.04715) (end 150.911 91.44715) (width 0.3) (layer F.Cu) (net 1))
+  (segment (start 150.52585 89.662) (end 150.911 90.04715) (width 0.3) (layer F.Cu) (net 1))
+  (segment (start 146.1135 89.662) (end 150.52585 89.662) (width 0.3) (layer F.Cu) (net 1))
+  (segment (start 150.911 92.84715) (end 150.911 91.44715) (width 0.3) (layer F.Cu) (net 1))
+  (segment (start 149.460999 94.297151) (end 150.911 92.84715) (width 0.3) (layer F.Cu) (net 1))
+  (segment (start 149.460999 99.842199) (end 149.460999 94.297151) (width 0.3) (layer F.Cu) (net 1))
+  (segment (start 150.911 101.2922) (end 149.460999 99.842199) (width 0.3) (layer F.Cu) (net 1))
+  (segment (start 150.911 102.6922) (end 150.911 101.2922) (width 0.3) (layer F.Cu) (net 1))
+  (segment (start 167.3695 108.377287) (end 167.3695 109.7915) (width 0.25) (layer B.Cu) (net 2))
+  (segment (start 167.3695 104.923809) (end 167.3695 108.377287) (width 0.3) (layer B.Cu) (net 2) (status 40000))
+  (segment (start 161.071 98.625309) (end 167.3695 104.923809) (width 0.3) (layer B.Cu) (net 2))
+  (segment (start 161.071 97.069675) (end 161.071 98.625309) (width 0.25) (layer B.Cu) (net 2) (status 40000))
+  (segment (start 161.071 95.514041) (end 162.9283 93.656741) (width 0.3) (layer B.Cu) (net 2))
+  (segment (start 161.071 97.069675) (end 161.071 95.514041) (width 0.3) (layer B.Cu) (net 2))
+  (segment (start 162.9283 87.681925) (end 161.071 85.824625) (width 0.3) (layer B.Cu) (net 2))
+  (segment (start 162.9283 93.656741) (end 162.9283 87.681925) (width 0.3) (layer B.Cu) (net 2))
+  (segment (start 161.071 80.6021) (end 161.371 80.3021) (width 0.3) (layer B.Cu) (net 2))
+  (segment (start 161.071 85.824625) (end 161.071 80.6021) (width 0.3) (layer B.Cu) (net 2))
+  (segment (start 162.3354 79.3377) (end 162.3354 76.8477) (width 0.3) (layer B.Cu) (net 2))
+  (segment (start 161.371 80.3021) (end 162.3354 79.3377) (width 0.3) (layer B.Cu) (net 2))
+  (segment (start 162.3354 76.8477) (end 164.8754 76.8477) (width 0.3) (layer B.Cu) (net 2))
+  (segment (start 162.3354 76.8477) (end 149.9275 76.8477) (width 0.3) (layer B.Cu) (net 2))
+  (segment (start 149.9275 76.8477) (end 147.3875 76.8477) (width 0.3) (layer B.Cu) (net 2))
+  (segment (start 149.9275 121.8311) (end 162.3989 121.8311) (width 0.3) (layer B.Cu) (net 2))
+  (segment (start 162.3989 121.8311) (end 164.9389 121.8311) (width 0.3) (layer B.Cu) (net 2))
+  (segment (start 167.3695 119.4005) (end 164.9389 121.8311) (width 0.3) (layer B.Cu) (net 2))
+  (segment (start 167.3695 109.7915) (end 167.3695 119.4005) (width 0.3) (layer B.Cu) (net 2))
+  (segment (start 144.8135 87.122) (end 146.1135 87.122) (width 0.3) (layer B.Cu) (net 2))
+  (segment (start 144.0942 87.8413) (end 144.8135 87.122) (width 0.3) (layer B.Cu) (net 2))
+  (segment (start 144.0942 97.3775) (end 144.0942 87.8413) (width 0.3) (layer B.Cu) (net 2))
+  (segment (start 146.4371 99.7204) (end 144.0942 97.3775) (width 0.3) (layer B.Cu) (net 2))
+  (segment (start 144.4371 98.8204) (end 143.2433 97.6266) (width 0.3) (layer F.Cu) (net 3))
+  (segment (start 144.4371 99.7204) (end 144.4371 98.8204) (width 0.3) (layer F.Cu) (net 3))
+  (segment (start 146.066 84.582) (end 146.1135 84.582) (width 0.3) (layer F.Cu) (net 3))
+  (segment (start 143.2433 87.4047) (end 146.066 84.582) (width 0.3) (layer F.Cu) (net 3))
+  (segment (start 143.2433 97.6266) (end 143.2433 87.4047) (width 0.3) (layer F.Cu) (net 3))
+  (segment (start 163.327699 84.754699) (end 165.0873 86.5143) (width 0.3) (layer F.Cu) (net 3))
+  (segment (start 163.327699 79.152099) (end 163.327699 84.754699) (width 0.3) (layer F.Cu) (net 3))
+  (segment (start 150.290901 79.152099) (end 151.656399 79.152099) (width 0.3) (layer F.Cu) (net 3))
+  (segment (start 146.1135 83.3295) (end 150.290901 79.152099) (width 0.3) (layer F.Cu) (net 3))
+  (segment (start 146.1135 84.582) (end 146.1135 83.3295) (width 0.3) (layer F.Cu) (net 3))
+  (segment (start 151.467201 79.152099) (end 151.656399 79.152099) (width 0.3) (layer F.Cu) (net 3))
+  (segment (start 151.656399 79.152099) (end 163.327699 79.152099) (width 0.3) (layer F.Cu) (net 3))
+  (segment (start 161.071 104.247834) (end 161.071 102.6922) (width 0.3) (layer B.Cu) (net 4))
+  (segment (start 161.071 106.448) (end 161.071 104.247834) (width 0.3) (layer B.Cu) (net 4))
+  (segment (start 156.7242 110.7948) (end 161.071 106.448) (width 0.3) (layer B.Cu) (net 4))
+  (segment (start 155.5242 110.7948) (end 156.7242 110.7948) (width 0.3) (layer B.Cu) (net 4))
+  (segment (start 155.448475 97.069675) (end 161.071 102.6922) (width 0.3) (layer F.Cu) (net 4))
+  (segment (start 150.911 97.069675) (end 155.448475 97.069675) (width 0.3) (layer F.Cu) (net 4))
+  (segment (start 150.911 87.224625) (end 150.911 85.824625) (width 0.3) (layer B.Cu) (net 5))
+  (segment (start 155.133525 91.44715) (end 150.911 87.224625) (width 0.3) (layer B.Cu) (net 5))
+  (segment (start 156.3116 91.4654) (end 156.32985 91.44715) (width 0.3) (layer B.Cu) (net 5))
+  (segment (start 156.3116 96.07955) (end 156.3116 91.4654) (width 0.3) (layer B.Cu) (net 5))
+  (segment (start 156.32985 91.44715) (end 155.133525 91.44715) (width 0.3) (layer B.Cu) (net 5))
+  (segment (start 149.7242 110.7948) (end 150.9242 110.7948) (width 0.3) (layer B.Cu) (net 5))
+  (segment (start 150.9242 110.7948) (end 156.3751 105.3439) (width 0.3) (layer B.Cu) (net 5))
+  (segment (start 156.3751 105.3439) (end 156.3751 96.14305) (width 0.3) (layer B.Cu) (net 5))
+  (segment (start 161.071 91.44715) (end 156.32985 91.44715) (width 0.3) (layer B.Cu) (net 5))
+  (segment (start 156.3751 96.14305) (end 156.3116 96.07955) (width 0.3) (layer B.Cu) (net 5))
+  (segment (start 165.5002 98.7552) (end 163.4109 96.6659) (width 0.3) (layer F.Cu) (net 6))
+  (segment (start 166.7002 98.7552) (end 165.5002 98.7552) (width 0.3) (layer F.Cu) (net 6))
+  (segment (start 163.4109 96.6659) (end 163.4109 91.641048) (width 0.3) (layer F.Cu) (net 6))
+  (segment (start 163.4109 91.641048) (end 163.4109 90.4621) (width 0.3) (layer F.Cu) (net 6))
+  (segment (start 153.751 81.43347) (end 153.751 80.3021) (width 0.3) (layer F.Cu) (net 6))
+  (segment (start 162.77963 90.4621) (end 153.751 81.43347) (width 0.3) (layer F.Cu) (net 6))
+  (segment (start 163.4109 90.4621) (end 162.77963 90.4621) (width 0.3) (layer F.Cu) (net 6))
+  (segment (start 149.9275 74.3077) (end 162.3354 74.3077) (width 0.3) (layer F.Cu) (net 7))
+  (segment (start 164.8754 74.3077) (end 162.3354 74.3077) (width 0.3) (layer F.Cu) (net 7))
+  (segment (start 149.9275 74.3077) (end 147.3875 74.3077) (width 0.3) (layer F.Cu) (net 7))
+  (segment (start 149.9275 119.2911) (end 162.3989 119.2911) (width 0.3) (layer F.Cu) (net 7))
+  (segment (start 162.3989 119.2911) (end 164.9389 119.2911) (width 0.3) (layer F.Cu) (net 7))
+  (segment (start 149.9275 119.2911) (end 147.3875 119.2911) (width 0.3) (layer F.Cu) (net 7))
+  (segment (start 166.075401 83.026199) (end 166.075401 75.486301) (width 0.3) (layer F.Cu) (net 7))
+  (segment (start 165.0873 84.0143) (end 166.075401 83.026199) (width 0.3) (layer F.Cu) (net 7))
+  (segment (start 166.054001 75.486301) (end 164.8754 74.3077) (width 0.3) (layer F.Cu) (net 7))
+  (segment (start 166.075401 75.486301) (end 166.054001 75.486301) (width 0.3) (layer F.Cu) (net 7))
+  (segment (start 166.7002 94.942408) (end 166.8145 94.828108) (width 0.3) (layer F.Cu) (net 7))
+  (segment (start 166.7002 96.2152) (end 166.7002 94.942408) (width 0.3) (layer F.Cu) (net 7))
+  (segment (start 166.8145 85.7415) (end 165.0873 84.0143) (width 0.3) (layer F.Cu) (net 7))
+  (segment (start 166.8145 94.828108) (end 166.8145 85.7415) (width 0.3) (layer F.Cu) (net 7))
+  (segment (start 164.9389 119.2911) (end 168.719501 115.510499) (width 0.3) (layer F.Cu) (net 7))
+  (segment (start 168.719501 115.510499) (end 168.719501 98.234501) (width 0.3) (layer F.Cu) (net 7))
+  (segment (start 168.719501 98.234501) (end 166.7002 96.2152) (width 0.3) (layer F.Cu) (net 7))
 )
