File: BreadBoard PS Variable/BreadBoard PS Variable/BreadBoard PS Variable.sch (KiCad schematic (older format))
At the start: 15 parts, among them J1 Barrel_Jack_Switch_MountingPin, J2 Conn_02x02_Odd_Even, J3 Conn_02x02_Odd_Even, J4 Conn_02x02_Odd_Even, J5 Conn_02x02_Odd_Even, SW1 SW_DPDT_x2, U1 LM7805_TO220

Commit message: Schematic
Parts:
- removed U1: LM7805_TO220, Package_TO_SOT_THT:TO-220-3_Vertical, symbol Regulator_Linear:LM7805_TO220
- added R?: 240Ω, Resistor_THT:R_Axial_DIN0207_L6.3mm_D2.5mm_P7.62mm_Horizontal, symbol Device:R_Small_US
- added RV?: R_POT_US, symbol Device:R_POT_US
- added U?: LM317T, digikey-footprints:TO-220-3, symbol dk_PMIC-Voltage-Regulators-Linear:LM317T
Connections:
- net Gnd: now also RV?.3
- net Vin: now also U?.3 (IN)
- net 5V renamed Vari-V
- net Vari-V: now also R?.1, U?.2 (OUT)
- net 5V-out renamed VariV-out
- new net: R?.2, RV?.1, RV?.2, U?.1 (ADJ)
Other:
- note added: "Vari-V Connectors"
- note added: "Variable V Regulator"
- note removed: "5V Connectors"
- note removed: "5V Regulator"
- moved on the sheet: C1, C2, D1, D2, D3, D4, D5, J1, J2, J3, J4, J5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
