File: BreadBoard PS Variable/BreadBoard PS Variable.kicad_pcb (KiCad board)
At the start: 2 copper layers, 29.8 x 52 mm, 19 parts, among them J1 Barrel_Jack_Switch_MountingPin, J2 Conn_02x02_Odd_Even, J3 Conn_02x02_Odd_Even, J4 Conn_02x02_Odd_Even, J5 Conn_02x02_Odd_Even, SW1 SW_SPDT, U1 LM317T

Commit message: PCB
Other:
- board text added: "Breadboard PS Variable Timothy S Leishman 12/8/21"
- board text removed: "Breadboard PS Variable Timothy S Leishman 12/7/21"
Changed lines of the file:
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@@
     (effects (font (size 1 1) (thickness 0.15)))
   )
-  (gr_text "Breadboard PS Variable\nTimothy S Leishman 12/7/21\n" (at 143.5608 100.6475 90) (layer B.SilkS)
+  (gr_text "Breadboard PS Variable\nTimothy S Leishman 12/8/21\n" (at 143.5608 100.6475 90) (layer B.SilkS)
     (effects (font (size 1 1) (thickness 0.15)) (justify left mirror))
   )
